File: hw/boards/shakesense-trenz-hat/pi-trenz-stack-concept.kicad_pcb (KiCad board)
At the start: 6 copper layers, 85 x 56 mm, 98 parts, among them J1 Raspberry Pi 40-pin, J2 Passive GNSS antenna, J4 FPGA test UART/reset, J80 LSHM-150-04.0-L-DV-A-S-K-TR, J81 LSHM-150-04.0-L-DV-A-S-K-TR, J82 LSHM-130-04.0-L-DV-A-S-K-TR, J83 1715721, J84 TSW-106-07-G-S, J85 TSW-103-07-G-D, Q1 2N7002, U1 24LC32A, U11 LSM6DSOTR, U12 LSM6DSOTR, U13 LSM6DSOTR, U14 LSM6DSOTR, U20 SCL3300-D01, U21 MAX-M10S, U40 TLV1117LV33DCYR, U41 SN74LVC8T245PWR, U42 SN74LVC8T245PWR, U43 ISO1640BDR, U51 TXU0202DCUR, U52 TLV803EA30DBZR

Commit message: Expose Trenz GPIOs on the Pi-outline HDI sensor HAT
Parts:
- added J86: BANK13 / 40p FFC, ShakeSense:TZ_FFC40, B.Cu at (67.0, 72.0)
- added J87: BANK14 / 40p FFC, ShakeSense:TZ_FFC40, B.Cu at (67.0, 89.0)
- added J88: BANK15 / 60p FFC, ShakeSense:TZ_FFC60, B.Cu at (107.0, 70.0)
- added J89: BANK16 / 60p FFC, ShakeSense:TZ_FFC60, B.Cu at (107.0, 87.0)
Connections:
- J80 pad 100: 100 -> FPGA_B14_L24_N
- J80 pad 11: GND -> 11
- J80 pad 15: 15 -> FPGA_B13_L6_N
- J80 pad 17: 17 -> FPGA_B13_L6_P
- J80 pad 18: 18 -> FPGA_B13_L3_P
- J80 pad 20: 20 -> FPGA_B13_L3_N
- J80 pad 21: 21 -> FPGA_B13_L5_N
- J80 pad 22: 22 -> FPGA_B13_L11_N
- J80 pad 23: 23 -> FPGA_B13_L5_P
- J80 pad 24: 24 -> FPGA_B13_L11_P
- J80 pad 25: 25 -> GND
- J80 pad 26: 26 -> FPGA_B13_L9_N
- J80 pad 28: 28 -> FPGA_B13_L9_P
- J80 pad 32: GND -> FPGA_B16_L22_P
- J80 pad 34: 34 -> FPGA_B16_L22_N
- J80 pad 35: j80-35 -> FPGA_B16_L16_P
- J80 pad 36: j80-36 -> FPGA_B16_L24_N
- J80 pad 37: 37 -> FPGA_B16_L16_N
- J80 pad 38: j80-38 -> FPGA_B16_L24_P
- J80 pad 39: 39 -> FPGA_B16_L19_N
- J80 pad 41: 41 -> FPGA_B16_L19_P
- J80 pad 42: 42 -> FPGA_B16_L23_P
- J80 pad 44: 44 -> FPGA_B16_L23_N
- J80 pad 45: 45 -> FPGA_B16_L17_N
- J80 pad 46: 46 -> FPGA_B16_L15_P
- J80 pad 47: 47 -> FPGA_B16_L17_P
- J80 pad 48: 48 -> FPGA_B16_L15_N
- J80 pad 49: 49 -> FPGA_B16_L18_N
- J80 pad 50: 50 -> FPGA_B16_L20_P
- J80 pad 51: 51 -> FPGA_B16_L18_P
- J80 pad 52: 52 -> FPGA_B16_L20_N
- J80 pad 55: 55 -> FPGA_B16_L9_N
- J80 pad 56: 56 -> FPGA_B16_L21_P
- J80 pad 57: 57 -> FPGA_B16_L9_P
- J80 pad 58: 58 -> FPGA_B16_L21_N
- J80 pad 59: 59 -> FPGA_B16_L7_N
- J80 pad 60: 60 -> FPGA_B16_L13_P
- J80 pad 61: 61 -> FPGA_B16_L7_P
- J80 pad 62: 62 -> FPGA_B16_L13_N
- J80 pad 65: 65 -> FPGA_B16_L11_P
- J80 pad 66: 66 -> FPGA_B16_L14_P
- J80 pad 67: 67 -> FPGA_B16_L11_N
- J80 pad 68: 68 -> FPGA_B16_L14_N
- J80 pad 69: 69 -> FPGA_B16_L10_N
- J80 pad 7: 7 -> GND
- J80 pad 70: 70 -> FPGA_B16_L3_N
- J80 pad 71: 71 -> FPGA_B16_L10_P
- J80 pad 72: 72 -> FPGA_B16_L3_P
- J80 pad 75: 75 -> FPGA_B16_L5_N
- J80 pad 76: 76 -> FPGA_B16_L12_P
- J80 pad 77: 77 -> FPGA_B16_L5_P
- J80 pad 78: 78 -> FPGA_B16_L12_N
- J80 pad 79: 79 -> FPGA_B16_L2_N
- J80 pad 81: 81 -> FPGA_B16_L2_P
- J80 pad 82: 82 -> FPGA_B16_L8_N
- J80 pad 83: 83 -> GND
- J80 pad 84: 84 -> FPGA_B16_L8_P
- J80 pad 85: 85 -> FPGA_B16_L6_N
- J80 pad 86: 86 -> FPGA_B14_L18_N
- J80 pad 87: 87 -> FPGA_B16_L6_P
- J80 pad 88: 88 -> FPGA_B14_L18_P
- J80 pad 91: 91 -> FPGA_B14_L24_P
- J80 pad 92: 92 -> FPGA_B14_L9_P
- J80 pad 93: 93 -> FPGA_B16_L4_N
- J80 pad 94: 94 -> FPGA_B14_L9_N
- J80 pad 95: 95 -> FPGA_B16_L4_P
- J80 pad 96: 96 -> FPGA_B14_L4_P
- J80 pad 97: 97 -> FPGA_B16_L1_N
- J80 pad 98: 98 -> FPGA_B14_L4_N
- J80 pad 99: 99 -> FPGA_B16_L1_P
- J81 pad 20: j81-20 -> 20
- J81 pad 21: j81-21 -> FPGA_B14_L12_P
- J81 pad 22: j81-22 -> FPGA_B14_L14_P
- J81 pad 23: j81-23 -> FPGA_B14_L12_N
- J81 pad 24: j81-24 -> FPGA_B14_L14_N
- J81 pad 25: j81-25 -> FPGA_B14_L11_P
- J81 pad 26: j81-26 -> FPGA_B14_L13_P
- J81 pad 27: 27 -> FPGA_B14_L11_N
- J81 pad 28: j81-28 -> FPGA_B14_L13_N
- J81 pad 29: GND -> 29
- J81 pad 30: GND -> 30
- J81 pad 31: 31 -> FPGA_B15_L9_N
- J81 pad 32: j81-32 -> FPGA_B14_L16_P
- J81 pad 33: 33 -> FPGA_B15_L9_P
- J81 pad 34: j81-34 -> FPGA_B14_L16_N
- J81 pad 35: j81-35 -> FPGA_B15_L8_N
- J81 pad 36: j81-36 -> FPGA_B14_L15_P
- J81 pad 37: j81-37 -> FPGA_B15_L8_P
- J81 pad 38: j81-38 -> FPGA_B14_L15_N
- J81 pad 41: j81-41 -> FPGA_B15_L7_N
- J81 pad 42: j81-42 -> FPGA_B15_L23_P
- J81 pad 43: 43 -> FPGA_B15_L7_P
- J81 pad 44: j81-44 -> FPGA_B15_L23_N
- J81 pad 45: j81-45 -> FPGA_B15_L13_P
- J81 pad 46: j81-46 -> FPGA_B15_L19_P
- J81 pad 47: j81-47 -> FPGA_B15_L13_N
- J81 pad 48: j81-48 -> FPGA_B15_L19_N
- J81 pad 51: j81-51 -> FPGA_B15_L14_P
- J81 pad 52: j81-52 -> FPGA_B15_L11_P
- J81 pad 53: 53 -> FPGA_B15_L14_N
- J81 pad 54: 54 -> FPGA_B15_L11_N
- J81 pad 55: j81-55 -> FPGA_B15_L12_P
- J81 pad 56: j81-56 -> FPGA_B15_L3_P
- J81 pad 57: j81-57 -> FPGA_B15_L12_N
- J81 pad 58: j81-58 -> FPGA_B15_L3_N
- J81 pad 61: j81-61 -> FPGA_B15_L10_N
- J81 pad 62: j81-62 -> FPGA_B15_L17_N
- J81 pad 63: 63 -> FPGA_B15_L10_P
- J81 pad 64: 64 -> FPGA_B15_L17_P
- J81 pad 65: j81-65 -> FPGA_B15_L18_P
- J81 pad 66: j81-66 -> FPGA_B15_L16_P
- J81 pad 67: j81-67 -> FPGA_B15_L18_N
- J81 pad 68: j81-68 -> FPGA_B15_L16_N
- J81 pad 71: j81-71 -> FPGA_B15_L20_P
- J81 pad 72: j81-72 -> FPGA_B15_L1_P
- J81 pad 73: 73 -> FPGA_B15_L20_N
- J81 pad 74: 74 -> FPGA_B15_L1_N
- J81 pad 75: j81-75 -> FPGA_B15_L15_P
- J81 pad 76: j81-76 -> FPGA_B15_L2_N
- J81 pad 77: j81-77 -> FPGA_B15_L15_N
- J81 pad 78: j81-78 -> FPGA_B15_L2_P
- J81 pad 81: j81-81 -> FPGA_B15_L6_N
- J81 pad 82: j81-82 -> FPGA_B15_L4_P
- J81 pad 83: j81-83 -> FPGA_B15_L6_P
- J81 pad 84: j81-84 -> FPGA_B15_L4_N
- J81 pad 85: j81-85 -> FPGA_B15_L21_P
- J81 pad 86: j81-86 -> FPGA_B15_L5_N
- J81 pad 87: j81-87 -> FPGA_B15_L21_N
- J81 pad 88: j81-88 -> FPGA_B15_L5_P
- J81 pad 90: 90 -> FPGA_B15_IO0
- J81 pad 91: j81-91 -> FPGA_B15_L24_N
- J81 pad 93: j81-93 -> FPGA_B15_L24_P
- J81 pad 95: j81-95 -> FPGA_B15_L22_N
- J81 pad 97: j81-97 -> FPGA_B15_L22_P
- J81 pad 99: j81-99 -> FPGA_B15_IO25
- J82 pad 1: 1 -> FPGA_B13_L14_P
- J82 pad 15: j82-15 -> 15
- J82 pad 2: 2 -> FPGA_B13_L17_P
- J82 pad 21: j82-21 -> 21
- J82 pad 22: j82-22 -> 22
- J82 pad 25: j82-25 -> 25
- J82 pad 26: j82-26 -> 26
- J82 pad 27: j82-27 -> 27
- J82 pad 28: j82-28 -> 28
- J82 pad 3: j82-3 -> FPGA_B13_L14_N
- J82 pad 31: j82-31 -> 31
- J82 pad 33: j82-33 -> 33
- J82 pad 34: j82-34 -> 34
- J82 pad 37: j82-37 -> FPGA_B13_L16_P
- J82 pad 38: j82-38 -> FPGA_B13_L10_P
- J82 pad 39: j82-39 -> FPGA_B13_L16_N
- J82 pad 4: 4 -> FPGA_B13_L17_N
- J82 pad 40: j82-40 -> FPGA_B13_L10_N
- J82 pad 41: j82-41 -> FPGA_B13_L1_P
- J82 pad 42: j82-42 -> FPGA_B13_L15_P
- J82 pad 43: j82-43 -> FPGA_B13_L1_N
- J82 pad 44: j82-44 -> FPGA_B13_L15_N
- J82 pad 47: j82-47 -> FPGA_B13_L4_P
- J82 pad 48: j82-48 -> FPGA_B14_L5_P
- J82 pad 49: j82-49 -> FPGA_B13_L4_N
- J82 pad 50: j82-50 -> FPGA_B14_L5_N
- J82 pad 51: j82-51 -> FPGA_B13_L2_N
- J82 pad 52: j82-52 -> FPGA_B14_L20_P
- J82 pad 53: j82-53 -> FPGA_B13_L2_P
- J82 pad 54: j82-54 -> FPGA_B14_L20_N
- J82 pad 55: j82-55 -> 55
- J82 pad 56: j82-56 -> 56
- J82 pad 57: j82-57 -> FPGA_B13_L12_P
- J82 pad 58: j82-58 -> FPGA_B13_L13_P
- J82 pad 59: j82-59 -> FPGA_B13_L12_N
- J82 pad 60: j82-60 -> FPGA_B13_L13_N
- J82 pad 7: j82-7 -> 7
- U11 pad 11: 11 -> u11-11
- U21 pad 18: u21-18 -> 18
- U21 pad 2: u21-2 -> 2
Routing:
- net GND: track 669.3 -> 873.3 mm, vias 1 -> 5
- net FPGA_B14_L24_P: track 0.00 -> 73.6 mm, vias 0 -> 2
- net FPGA_B14_L24_N: track 0.00 -> 66.8 mm, vias 0 -> 2
- net FPGA_3V3: track 163.0 -> 227.7 mm, vias 4 -> 6
- net FPGA_B14_L18_P: track 0.00 -> 60.1 mm, vias 0 -> 2
- net FPGA_B14_L18_N: track 0.00 -> 59.2 mm, vias 0 -> 2
- net FPGA_B14_L9_N: track 0.00 -> 58.3 mm, vias 0 -> 2
- net FPGA_B14_L14_P: track 0.00 -> 57.6 mm, vias 0 -> 3
- net FPGA_B14_L9_P: track 0.00 -> 57.4 mm, vias 0 -> 2
- net FPGA_B14_L16_N: track 0.00 -> 57.4 mm, vias 0 -> 3
- net FPGA_B13_L5_N: track 0.00 -> 57.1 mm, vias 0 -> 3
- net FPGA_B14_L16_P: track 0.00 -> 55.6 mm, vias 0 -> 3
- net FPGA_B13_L3_P: track 0.00 -> 55.1 mm, vias 0 -> 3
- net FPGA_B14_L4_P: track 0.00 -> 55.1 mm, vias 0 -> 2
- net FPGA_B14_L15_N: track 0.00 -> 54.8 mm, vias 0 -> 3
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- added copper zone on In2.Cu, net GND
- added copper zone on In5.Cu, net GND
- removed copper zone on In1.Cu, net GND
- removed copper zone on In4.Cu, net GND
Other:
- copper layers 6 -> 8
- board text added: "GPIO J86 B13 3V3"
- board text added: "GPIO J87 B14 3V3"
- board text added: "GPIO J88 B15 3V3"
- board text added: "GPIO J89 B16 3V3"
