File: hw/boards/shakesense-trenz-hat/03-geophone-page-01.kicad_sch (KiCad schematic)
At the start: 12 parts, among them J90 GEO + / - / SHIELD, U22 ADS122C04

Commit message: Harden geophone acquisition and tighten analog layout
Parts:
- C90: MPN C1206C104J5GACTU -> C3216C0G1H104J160AA
Changed lines of the file:
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@@
               (property "Value" "100n C0G" (at 147.32 79.78 0) (effects (font (size 1.0 1.0))))
               (property "Footprint" "ShakeSense:Capacitor_SMD__C_1206_3216Metric" (at 147.32 83.82000000000001 0) (effects (font (size 1 1)) hide))
-              (property "MPN" "C1206C104J5GACTU" (at 147.32 83.82000000000001 0) (effects (font (size 1 1)) hide))
+              (property "MPN" "C3216C0G1H104J160AA" (at 147.32 83.82000000000001 0) (effects (font (size 1 1)) hide))
               (instances (project "shakesense-trenz-hat" (path "/4ffaaa5d-c728-540d-9f0f-f1cafbdbe36e/0c18b12e-d7e6-548b-b124-7cc01c20072f" (reference "C90") (unit 1)))))
 (wire (pts (xy 132.08 83.82) (xy 127.0 83.82)) (stroke (width 0) (type default)))
