File: hw/boards/shakesense-trenz-hat/shakesense-trenz-hat.kicad_sch (KiCad schematic)
At the start: 0 parts

Commit message: Expose Trenz GPIOs on the Pi-outline HDI sensor HAT
Other:
- added sheet 11-gpio-bank13-page-01 (11-gpio-bank13-page-01.kicad_sch)
- added sheet 11-gpio-bank14-page-01 (11-gpio-bank14-page-01.kicad_sch)
- added sheet 11-gpio-bank15-page-01 (11-gpio-bank15-page-01.kicad_sch)
- added sheet 11-gpio-bank16-page-01 (11-gpio-bank16-page-01.kicad_sch)
- note added: "Atopile-derived review schematic - T1 GPIO prototype, not released. Pi sensor acquisition; 155 expansion GPIOs at 3.3 V; Coldfoot integration deferred. Global net labels connect functional sheets."
- note removed: "Atopile-derived review schematic - prototype, not released. The Pi hosts acquisition and Coldfoot processing; the USB head has a local MCU. Global net labels connect functional sheets."

Commit message: Replace T1 GNSS with single Racotech geophone input
Other:
- added sheet 03-geophone-page-01 (03-geophone-page-01.kicad_sch)
- added sheet 03-geophone-page-02 (03-geophone-page-02.kicad_sch)
- note added: "Atopile-derived review schematic - T1 geophone / GPIO prototype, not released. Pi sensor acquisition; 155 expansion GPIOs at 3.3 V; Coldfoot integration deferred. Global net labels connect functional sheets."
- note removed: "Atopile-derived review schematic - T1 GPIO prototype, not released. Pi sensor acquisition; 155 expansion GPIOs at 3.3 V; Coldfoot integration deferred. Global net labels connect functional sheets."

Commit message: Implement internal Pi FPGA link and remove ribbon expansion
Other:
- removed sheet 11-gpio-bank13-page-01
- removed sheet 11-gpio-bank14-page-01
- removed sheet 11-gpio-bank15-page-01
- removed sheet 11-gpio-bank16-page-01
- added sheet 07-internal-link-page-01 (07-internal-link-page-01.kicad_sch)
- added sheet 07-internal-link-page-02 (07-internal-link-page-02.kicad_sch)
- added sheet 07-internal-link-page-03 (07-internal-link-page-03.kicad_sch)
- note added: "Atopile-derived review schematic - T1 geophone / internal-link prototype, not released. Pi sensor acquisition; SPI6 / quad wiring, UART and switched Pi JTAG; Coldfoot integration deferred. Global net labels connect functional sheets."
- note removed: "Atopile-derived review schematic - T1 geophone / GPIO prototype, not released. Pi sensor acquisition; 155 expansion GPIOs at 3.3 V; Coldfoot integration deferred. Global net labels connect functional sheets."
