File: hw/boards/shakesense-trenz-hat/stack-service-envelopes.kicad_pcb (KiCad board)
At the start: 8 copper layers, 85 x 56 mm, 116 parts, among them J1 Raspberry Pi 40-pin, J4 FPGA test UART/reset, J80 LSHM-150-04.0-L-DV-A-S-K-TR, J81 LSHM-150-04.0-L-DV-A-S-K-TR, J82 LSHM-130-04.0-L-DV-A-S-K-TR, J83 1715721, J84 TSW-106-07-G-S, J85 TSW-103-07-G-D, J86 BANK13 / 40p FFC, J87 BANK14 / 40p FFC, J88 BANK15 / 60p FFC, J89 BANK16 / 60p FFC, J90 GEO + / - / SHIELD, Q1 2N7002, U1 24LC32A, U11 LSM6DSOTR, U12 LSM6DSOTR, U13 LSM6DSOTR, U14 LSM6DSOTR, U20 SCL3300-D01, U22 ADS122C04, U40 TLV1117LV33DCYR, U41 SN74LVC8T245PWR, U42 SN74LVC8T245PWR, U43 ISO1640BDR, U51 TXU0202DCUR, U52 TLV803EA30DBZR

Commit message: Resolve T1 ribbon clearance with guided flex and windowed support
Parts:
- added MODEL_OFFSET_SPACER, MODEL_RIBBONS, MODEL_RIBBON_GUIDE: Visualization only, , F.Cu at (50.0, 50.0)
- moved J87 3.00 mm to (67.0, 86.0)
- moved J83 2.30 mm to (54.7, 62.0)
Routing:
- net GND: track 813.0 -> 868.5 mm, vias 18 -> 30
- net FPGA_B14_L4_N: track 49.4 -> 82.5 mm, vias 3 -> 7
- net FPGA_B13_L6_P: track 44.1 -> 59.4 mm
- net FPGA_B14_L4_P: track 49.6 -> 64.1 mm, vias 2 -> 4
- net FPGA_3V3: track 227.7 -> 241.5 mm, vias 6 -> 8
- net FPGA_B14_L11_P: track 42.6 -> 53.5 mm, vias 3 -> 5
- net FPGA_B14_L5_P: track 22.1 -> 31.4 mm
- net FPGA_B13_L3_P: track 51.8 -> 60.8 mm, vias 6 -> 5
- net FPGA_B14_L14_P: track 57.6 -> 48.9 mm, vias 3 -> 5
- net FPGA_B14_L18_N: track 59.2 -> 66.7 mm, vias 2 -> 5
- net FPGA_B14_L18_P: track 107.0 -> 112.0 mm, vias 4 -> 6
- net FPGA_B14_L9_N: track 58.3 -> 62.2 mm
- net FPGA_B14_L9_P: track 57.4 -> 61.2 mm
- net FPGA_B14_L24_N: track 66.8 -> 70.3 mm
- net FPGA_B14_L15_P: track 53.5 -> 50.1 mm
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
Commit message: Implement internal Pi FPGA link and remove ribbon expansion
Parts:
- removed J84: TSW-106-07-G-S, ShakeSense:TZ_TZ_JTAG
- removed J85: TSW-103-07-G-D, ShakeSense:TZ_TZ_AUX
- removed J86: BANK13 / 40p FFC, ShakeSense:TZ_FFC40
- removed J87: BANK14 / 40p FFC, ShakeSense:TZ_FFC40
- removed J88: BANK15 / 60p FFC, ShakeSense:TZ_FFC60
- removed J89: BANK16 / 60p FFC, ShakeSense:TZ_FFC60
- removed MODEL_OFFSET_SPACER, MODEL_RIBBONS, MODEL_RIBBON_GUIDE: Visualization only, 
- added C100: 100n, ShakeSense:Capacitor_SMD__C_0603_1608Metric, B.Cu at (106.0, 69.7)
- added C101: 100n, ShakeSense:Capacitor_SMD__C_0603_1608Metric, B.Cu at (106.0, 81.7)
- added C102: 100n, ShakeSense:Capacitor_SMD__C_0603_1608Metric, B.Cu at (73.0, 69.7)
- added C103: 100n, ShakeSense:Capacitor_SMD__C_0603_1608Metric, B.Cu at (84.8, 71.7)
- added C104: 100n, ShakeSense:Capacitor_SMD__C_0603_1608Metric, B.Cu at (77.5, 80.0)
- added C105: 100n, ShakeSense:Capacitor_SMD__C_0603_1608Metric, B.Cu at (84.5, 80.0)
- added C106: , ShakeSense:Capacitor_SMD__C_0603_1608Metric, B.Cu at (79.0, 90.0)
- added R100: 22, ShakeSense:Resistor_SMD__R_0603_1608Metric, B.Cu at (99.0, 58.0)
- added R101: 22, ShakeSense:Resistor_SMD__R_0603_1608Metric, B.Cu at (94.0, 58.0)
- added R102: 22, ShakeSense:Resistor_SMD__R_0603_1608Metric, B.Cu at (89.0, 58.0)
- added R103: 22, ShakeSense:Resistor_SMD__R_0603_1608Metric, B.Cu at (84.0, 58.0)
- added R104: 22, ShakeSense:Resistor_SMD__R_0603_1608Metric, B.Cu at (79.0, 58.0)
- added R105: 22, ShakeSense:Resistor_SMD__R_0603_1608Metric, B.Cu at (74.0, 58.0)
- added R106: 10k, ShakeSense:Resistor_SMD__R_0603_1608Metric, B.Cu at (79.0, 68.0)
- added R107: 10k, ShakeSense:Resistor_SMD__R_0603_1608Metric, B.Cu at (79.0, 70.0)
- added R108: 10k, ShakeSense:Resistor_SMD__R_0603_1608Metric, B.Cu at (88.0, 72.0)
- added R109: 10k, ShakeSense:Resistor_SMD__R_0603_1608Metric, B.Cu at (74.0, 83.0)
- added R110: 10k, ShakeSense:Resistor_SMD__R_0603_1608Metric, B.Cu at (81.0, 83.0)
- added R111: 10k, ShakeSense:Resistor_SMD__R_0603_1608Metric, B.Cu at (94.0, 81.0)
- added R112: 100k, ShakeSense:Resistor_SMD__R_0603_1608Metric, B.Cu at (94.0, 69.0)
- added R113: 10k, ShakeSense:Resistor_SMD__R_0603_1608Metric, B.Cu at (94.0, 75.0)
- added R114: 100k, ShakeSense:Resistor_SMD__R_0603_1608Metric, B.Cu at (94.0, 71.0)
- added R115: 10k, ShakeSense:Resistor_SMD__R_0603_1608Metric, B.Cu at (94.0, 73.0)
- added R116: 100k, ShakeSense:Resistor_SMD__R_0603_1608Metric, B.Cu at (106.0, 75.0)
- added R117: 100k, ShakeSense:Resistor_SMD__R_0603_1608Metric, B.Cu at (94.0, 85.0)
- added U100: TMUX1574PWR, ShakeSense:Package_SO__TSSOP-16_4.4x5mm_P0.65mm, B.Cu at (100.0, 72.0)
- added U101: TMUX1574PWR, ShakeSense:Package_SO__TSSOP-16_4.4x5mm_P0.65mm, B.Cu at (100.0, 84.0)
- added U102: TCA9534PWR, ShakeSense:Package_SO__TSSOP-16_4.4x5mm_P0.65mm, B.Cu at (67.0, 72.0)
- added U103: SN74LVC1G10DCKR, ShakeSense:Package_TO_SOT_SMD__SOT-363_SC-70-6, B.Cu at (81.0, 72.0)
- added U104: TLV809EA30DBZR, ShakeSense:Package_TO_SOT_SMD__SOT-23, B.Cu at (74.0, 80.0)
- added U105: TLV809EA30DBZR, ShakeSense:Package_TO_SOT_SMD__SOT-23, B.Cu at (81.0, 80.0)
- added U106: , ShakeSense:Package_TO_SOT_SMD__SOT-353_SC-70-5, B.Cu at (75.5, 90.0)
Connections:
- J1 pad 12: 12 -> PI_LINK_CS_N
- J1 pad 32: 32 -> PI_LINK_DQ3
- J1 pad 35: 35 -> PI_LINK_DQ1
- J1 pad 36: 36 -> PI_LINK_DQ2
- J1 pad 38: 38 -> PI_LINK_DQ0
- J1 pad 40: 40 -> PI_LINK_SCLK
- J80 pad 100: FPGA_B14_L24_N -> 100
- J80 pad 15: FPGA_B13_L6_N -> 15
- J80 pad 17: FPGA_B13_L6_P -> 17
- J80 pad 18: FPGA_B13_L3_P -> 18
- J80 pad 20: FPGA_B13_L3_N -> 20
- J80 pad 21: FPGA_B13_L5_N -> 21
- J80 pad 22: FPGA_B13_L11_N -> 22
- J80 pad 23: FPGA_B13_L5_P -> 23
- J80 pad 24: FPGA_B13_L11_P -> 24
- J80 pad 26: FPGA_B13_L9_N -> 26
- J80 pad 28: FPGA_B13_L9_P -> 28
- J80 pad 32: FPGA_B16_L22_P -> 32
- J80 pad 34: FPGA_B16_L22_N -> 34
- J80 pad 35: FPGA_B16_L16_P -> 35
- J80 pad 36: FPGA_B16_L24_N -> 36
- J80 pad 37: FPGA_B16_L16_N -> 37
- J80 pad 38: FPGA_B16_L24_P -> 38
- J80 pad 39: FPGA_B16_L19_N -> 39
- J80 pad 40: j80-40 -> 40
- J80 pad 41: FPGA_B16_L19_P -> 41
- J80 pad 42: FPGA_B16_L23_P -> 42
- J80 pad 44: FPGA_B16_L23_N -> 44
- J80 pad 45: FPGA_B16_L17_N -> 45
- J80 pad 46: FPGA_B16_L15_P -> 46
- J80 pad 47: FPGA_B16_L17_P -> 47
- J80 pad 48: FPGA_B16_L15_N -> 48
- J80 pad 49: FPGA_B16_L18_N -> 49
- J80 pad 50: FPGA_B16_L20_P -> 50
- J80 pad 51: FPGA_B16_L18_P -> 51
- J80 pad 52: FPGA_B16_L20_N -> 52
- J80 pad 55: FPGA_B16_L9_N -> 55
- J80 pad 56: FPGA_B16_L21_P -> 56
- J80 pad 57: FPGA_B16_L9_P -> 57
- J80 pad 58: FPGA_B16_L21_N -> 58
- J80 pad 59: FPGA_B16_L7_N -> 59
- J80 pad 60: FPGA_B16_L13_P -> 60
- J80 pad 61: FPGA_B16_L7_P -> 61
- J80 pad 62: FPGA_B16_L13_N -> 62
- J80 pad 65: FPGA_B16_L11_P -> 65
- J80 pad 66: FPGA_B16_L14_P -> 66
- J80 pad 67: FPGA_B16_L11_N -> 67
- J80 pad 68: FPGA_B16_L14_N -> 68
- J80 pad 69: FPGA_B16_L10_N -> 69
- J80 pad 70: FPGA_B16_L3_N -> 70
- J80 pad 71: FPGA_B16_L10_P -> 71
- J80 pad 72: FPGA_B16_L3_P -> 72
- J80 pad 75: FPGA_B16_L5_N -> 75
- J80 pad 76: FPGA_B16_L12_P -> 76
- J80 pad 77: FPGA_B16_L5_P -> 77
- J80 pad 78: FPGA_B16_L12_N -> 78
- J80 pad 79: FPGA_B16_L2_N -> 79
- J80 pad 81: FPGA_B16_L2_P -> 81
- J80 pad 82: FPGA_B16_L8_N -> 82
- J80 pad 84: FPGA_B16_L8_P -> 84
- J80 pad 85: FPGA_B16_L6_N -> 85
- J80 pad 86: FPGA_B14_L18_N -> 86
- J80 pad 87: FPGA_B16_L6_P -> 87
- J80 pad 88: FPGA_B14_L18_P -> 88
- J80 pad 91: FPGA_B14_L24_P -> 91
- J80 pad 92: FPGA_B14_L9_P -> 92
- J80 pad 93: FPGA_B16_L4_N -> 93
- J80 pad 94: FPGA_B14_L9_N -> 94
- J80 pad 95: FPGA_B16_L4_P -> 95
- J80 pad 96: FPGA_B14_L4_P -> 96
- J80 pad 97: FPGA_B16_L1_N -> 97
- J80 pad 98: FPGA_B14_L4_N -> 98
- J80 pad 99: FPGA_B16_L1_P -> 99
- J81 pad 15: FPGA_AUX0 -> j81-15
- J81 pad 16: FPGA_AUX1 -> 16
- J81 pad 18: FPGA_AUX2 -> j81-18
- J81 pad 20: 20 -> j81-20
- J81 pad 21: FPGA_B14_L12_P -> FPGA_LINK_SCLK
- J81 pad 22: FPGA_B14_L14_P -> FPGA_LINK_DQ0
- J81 pad 23: FPGA_B14_L12_N -> FPGA_LINK_CS_N
- J81 pad 24: FPGA_B14_L14_N -> FPGA_LINK_DQ1
- J81 pad 25: FPGA_B14_L11_P -> 25
- J81 pad 26: FPGA_B14_L13_P -> FPGA_LINK_DQ2
- J81 pad 27: FPGA_B14_L11_N -> 27
- J81 pad 28: FPGA_B14_L13_N -> FPGA_LINK_DQ3
- J81 pad 31: FPGA_B15_L9_N -> 31
- J81 pad 32: FPGA_B14_L16_P -> j81-32
- J81 pad 33: FPGA_B15_L9_P -> 33
- J81 pad 34: FPGA_B14_L16_N -> j81-34
- J81 pad 35: FPGA_B15_L8_N -> j81-35
- J81 pad 36: FPGA_B14_L15_P -> j81-36
- J81 pad 37: FPGA_B15_L8_P -> j81-37
- J81 pad 38: FPGA_B14_L15_N -> j81-38
- J81 pad 41: FPGA_B15_L7_N -> j81-41
- J81 pad 42: FPGA_B15_L23_P -> j81-42
- J81 pad 43: FPGA_B15_L7_P -> 43
- J81 pad 44: FPGA_B15_L23_N -> j81-44
- J81 pad 45: FPGA_B15_L13_P -> j81-45
- J81 pad 46: FPGA_B15_L19_P -> j81-46
- J81 pad 47: FPGA_B15_L13_N -> j81-47
- J81 pad 48: FPGA_B15_L19_N -> j81-48
- J81 pad 51: FPGA_B15_L14_P -> j81-51
- J81 pad 52: FPGA_B15_L11_P -> j81-52
- J81 pad 53: FPGA_B15_L14_N -> 53
- J81 pad 54: FPGA_B15_L11_N -> 54
- J81 pad 55: FPGA_B15_L12_P -> j81-55
- J81 pad 56: FPGA_B15_L3_P -> j81-56
- J81 pad 57: FPGA_B15_L12_N -> j81-57
- J81 pad 58: FPGA_B15_L3_N -> j81-58
- J81 pad 61: FPGA_B15_L10_N -> j81-61
- J81 pad 62: FPGA_B15_L17_N -> j81-62
- J81 pad 63: FPGA_B15_L10_P -> 63
- J81 pad 64: FPGA_B15_L17_P -> 64
- J81 pad 65: FPGA_B15_L18_P -> j81-65
- J81 pad 66: FPGA_B15_L16_P -> j81-66
- J81 pad 67: FPGA_B15_L18_N -> j81-67
- J81 pad 68: FPGA_B15_L16_N -> j81-68
- J81 pad 71: FPGA_B15_L20_P -> j81-71
- J81 pad 72: FPGA_B15_L1_P -> j81-72
- J81 pad 73: FPGA_B15_L20_N -> 73
- J81 pad 74: FPGA_B15_L1_N -> 74
- J81 pad 75: FPGA_B15_L15_P -> j81-75
- J81 pad 76: FPGA_B15_L2_N -> j81-76
- J81 pad 77: FPGA_B15_L15_N -> j81-77
- J81 pad 78: FPGA_B15_L2_P -> j81-78
- J81 pad 81: FPGA_B15_L6_N -> j81-81
- J81 pad 82: FPGA_B15_L4_P -> j81-82
- J81 pad 83: FPGA_B15_L6_P -> 83
- J81 pad 84: FPGA_B15_L4_N -> j81-84
- J81 pad 85: FPGA_B15_L21_P -> j81-85
- J81 pad 86: FPGA_B15_L5_N -> j81-86
- J81 pad 87: FPGA_B15_L21_N -> j81-87
- J81 pad 88: FPGA_B15_L5_P -> j81-88
- J81 pad 90: FPGA_B15_IO0 -> 90
- J81 pad 91: FPGA_B15_L24_N -> j81-91
- J81 pad 93: FPGA_B15_L24_P -> j81-93
- J81 pad 95: FPGA_B15_L22_N -> j81-95
- J81 pad 97: FPGA_B15_L22_P -> j81-97
- J81 pad 99: FPGA_B15_IO25 -> j81-99
- J82 pad 1: FPGA_B13_L14_P -> 1
- J82 pad 15: 15 -> j82-15
- J82 pad 16: 16 -> j82-16
- J82 pad 2: FPGA_B13_L17_P -> 2
- J82 pad 21: 21 -> j82-21
- J82 pad 22: 22 -> j82-22
- J82 pad 25: 25 -> j82-25
- J82 pad 26: 26 -> j82-26
- J82 pad 27: 27 -> j82-27
- J82 pad 28: 28 -> j82-28
- J82 pad 3: FPGA_B13_L14_N -> j82-3
- J82 pad 31: 31 -> j82-31
- J82 pad 33: 33 -> j82-33
- J82 pad 34: 34 -> j82-34
- J82 pad 37: FPGA_B13_L16_P -> j82-37
- J82 pad 38: FPGA_B13_L10_P -> j82-38
- J82 pad 39: FPGA_B13_L16_N -> j82-39
- J82 pad 4: FPGA_B13_L17_N -> 4
- J82 pad 40: FPGA_B13_L10_N -> j82-40
- J82 pad 41: FPGA_B13_L1_P -> j82-41
- J82 pad 42: FPGA_B13_L15_P -> j82-42
- J82 pad 43: FPGA_B13_L1_N -> j82-43
- J82 pad 44: FPGA_B13_L15_N -> j82-44
- J82 pad 47: FPGA_B13_L4_P -> j82-47
- J82 pad 48: FPGA_B14_L5_P -> j82-48
- J82 pad 49: FPGA_B13_L4_N -> j82-49
- J82 pad 50: FPGA_B14_L5_N -> j82-50
- J82 pad 51: FPGA_B13_L2_N -> j82-51
- J82 pad 52: FPGA_B14_L20_P -> j82-52
- J82 pad 53: FPGA_B13_L2_P -> j82-53
- J82 pad 54: FPGA_B14_L20_N -> j82-54
- J82 pad 55: 55 -> j82-55
- J82 pad 56: 56 -> j82-56
- J82 pad 57: FPGA_B13_L12_P -> j82-57
- J82 pad 58: FPGA_B13_L13_P -> j82-58
- J82 pad 59: FPGA_B13_L12_N -> j82-59
- J82 pad 60: FPGA_B13_L13_N -> j82-60
Routing:
- net FPGA_B14_L18_P: track 112.0 -> 0.00 mm, vias 6 -> 0
- net GND: track 868.5 -> 781.2 mm, vias 30 -> 55
- net FPGA_B14_L4_N: track 82.5 -> 0.00 mm, vias 7 -> 0
- net FPGA_B14_L24_N: track 70.3 -> 0.00 mm, vias 2 -> 0
- net FPGA_B14_L24_P: track 68.4 -> 0.00 mm, vias 6 -> 0
- net FPGA_B14_L18_N: track 66.7 -> 0.00 mm, vias 5 -> 0
- net FPGA_B14_L4_P: track 64.1 -> 0.00 mm, vias 4 -> 0
- net LINK_JTAG_SEL: track 0.00 -> 62.8 mm, vias 0 -> 4
- net FPGA_B14_L9_N: track 62.2 -> 0.00 mm, vias 5 -> 0
- net FPGA_B14_L9_P: track 61.2 -> 0.00 mm, vias 2 -> 0
- net FPGA_B13_L3_P: track 60.8 -> 0.00 mm, vias 5 -> 0
- net FPGA_B13_L6_P: track 59.4 -> 0.00 mm, vias 5 -> 0
- net FPGA_B13_L5_N: track 57.1 -> 0.00 mm, vias 3 -> 0
- net FPGA_B14_L15_N: track 56.7 -> 0.00 mm, vias 5 -> 0
- net FPGA_AUX2: track 55.5 -> 0.00 mm, vias 1 -> 0
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Other:
- board text removed: "GPIO J86 B13 3V3"
- board text removed: "GPIO J87 B14 3V3"
- board text removed: "GPIO J88 B15 3V3"
- board text removed: "GPIO J89 B16 3V3"
- board text removed: "JTAG"
