File: hw/boards/shakesense-trenz-hat/shakesense-trenz-hat.kicad_pcb (KiCad board)
At the start: 8 copper layers, 85 x 56 mm, 138 parts, among them J1 Raspberry Pi 40-pin, J4 FPGA test UART/reset, J80 LSHM-150-04.0-L-DV-A-S-K-TR, J81 LSHM-150-04.0-L-DV-A-S-K-TR, J82 LSHM-130-04.0-L-DV-A-S-K-TR, J83 1715721, J90 GEO + / - / SHIELD, Q1 2N7002, U1 24LC32A, U100 TMUX1574PWR, U101 TMUX1574PWR, U102 TCA9534PWR, U103 SN74LVC1G10DCKR, U104 TLV809EA30DBZR, U105 TLV809EA30DBZR, U11 LSM6DSOTR, U12 LSM6DSOTR, U13 LSM6DSOTR, U14 LSM6DSOTR, U20 SCL3300-D01, U22 ADS122C04, U40 TLV1117LV33DCYR, U41 SN74LVC8T245PWR, U42 SN74LVC8T245PWR, U43 ISO1640BDR, U51 TXU0202DCUR, U52 TLV803EA30DBZR

Commit message: Harden T1 FPGA transport and expand pre-fab verification
Parts:
- C106: value (none) -> 100n
- U106: value (none) -> SN74LVC1G08DCKR
Changed lines of the file:
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@@
 			)
 		)
-		(property "Value" ""
+		(property "Value" "SN74LVC1G08DCKR"
 			(at 0 -1.95 180)
 			(layer "B.Fab")
@@
 			)
 		)
-		(property "Value" ""
+		(property "Value" "100n"
 			(at 0 -1.43 180)
 			(layer "B.Fab")
