File: hw/layout/field_head/field_head.kicad_pcb (KiCad board)
At the start: 2 copper layers, 27 parts

Commit message: Rename project to Groundlark and sensor carrier to DAQHAT-01
Parts:
- U2: footprint elec:ShakeSense__PNI_14190_Module -> elec:Groundlark__PNI_14190_Module
- U3: footprint elec:ShakeSense__DLVR_E1BS -> elec:Groundlark__DLVR_E1BS
Changed lines of the file:
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@@
 		)
 	)
-	(footprint "elec:ShakeSense__PNI_14190_Module"
+	(footprint "elec:Groundlark__PNI_14190_Module"
 		(layer "F.Cu")
 		(at 230 0 0)
@@
 		)
 	)
-	(footprint "elec:ShakeSense__DLVR_E1BS"
+	(footprint "elec:Groundlark__DLVR_E1BS"
 		(layer "F.Cu")
 		(at 250 0 0)
