File: hw/layout/hat/hat.kicad_pcb (KiCad board)
At the start: 2 copper layers, 143 parts

Commit message: Rename project to Groundlark and sensor carrier to DAQHAT-01
Parts:
- U20: footprint elec:ShakeSense__SCL3300_D01 -> elec:Groundlark__SCL3300_D01
Changed lines of the file:
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@@
 		)
 	)
-	(footprint "elec:ShakeSense__SCL3300_D01"
+	(footprint "elec:Groundlark__SCL3300_D01"
 		(layer "F.Cu")
 		(at 250 0)
