File: hw/boards/groundlark-daqhat-01/01-host-power-page-01.kicad_sch (KiCad schematic)
At the start: 9 parts, among them J1 Raspberry Pi 40-pin, U1 24LC32A

Commit message: Harden DAQHAT-01 assembly exports and refresh stack overview
Publish the current three-IMU six-layer revision and matching software. Capture exact-part sourcing, shortage substitutions and numbered-pad rotation mappings with regression and full/overlay integration tests. Preserve validated BOM bytes across Git checkouts. Replace README images with the current stack and a dimensioned geophone illustration; keep fabrication packages local.
Connections:
- net PI_IMU4_CS: no longer names the net of J1.31
- net PI_IMU4_INT: no longer names the net of J1.18
- net PI_TILT_CS: no longer names the net of J1.33
- no-connect marks 0 -> 3
