File: hw/boards/groundlark-daqhat-01/06-supply-isolation-page-01.kicad_sch (KiCad schematic)
At the start: 12 parts, among them U40 TLV1117LV33DCYR, U41 SN74LVC8T245PWR, U42 SN74LVC8T245PWR

Commit message: Harden DAQHAT-01 assembly exports and refresh stack overview
Publish the current three-IMU six-layer revision and matching software. Capture exact-part sourcing, shortage substitutions and numbered-pad rotation mappings with regression and full/overlay integration tests. Preserve validated BOM bytes across Git checkouts. Replace README images with the current stack and a dimensioned geophone illustration; keep fabrication packages local.
Connections:
- net IMU4_INT is gone; now on net GND: U42.17 (B5)
- net PI_IMU4_CS is gone; now on net GND: U41.8 (A6)
- net PI_TILT_CS is gone; now on net GND: U41.9 (A7)
- net IMU4_CS: no longer names the net of U41.16 (B6)
- net PI_IMU4_INT: no longer names the net of U42.7 (A5)
- net TILT_CS: no longer names the net of U41.15 (B7)
- no-connect marks 3 -> 6
