File: hw/boards/groundlark-daqhat-01/groundlark-daqhat-01.kicad_sch (KiCad schematic)
At the start: 0 parts

Commit message: Harden DAQHAT-01 assembly exports and refresh stack overview
Publish the current three-IMU six-layer revision and matching software. Capture exact-part sourcing, shortage substitutions and numbered-pad rotation mappings with regression and full/overlay integration tests. Preserve validated BOM bytes across Git checkouts. Replace README images with the current stack and a dimensioned geophone illustration; keep fabrication packages local.
Other:
- removed sheet 02-motion-array-page-02
- removed sheet 03-level-position-page-01
